File: cad/PCBs/Digit/Digit.kicad_sch (KiCad schematic)
At the start: 0 parts

Commit message: Initial Digit Schematic and Layout
Parts:
- added C1, C10, C11, C12, C13, C14, C2, C3, C4, C5, C6, C7, C8, C9: 0.1 uF, Capacitor_SMD:C_0805_2012Metric, symbol Device:C_Small
- added D2, D3: SS310, Diode_SMD:D_SOD-323F, symbol Device:D_Schottky_Small
- added J1: Digit_IN, Connector_PinHeader_2.54mm:PinHeader_1x06_P2.54mm_Horizontal, symbol Connector_Generic:Conn_01x06
- added J2: Digit_OUT, Connector_PinHeader_2.54mm:PinHeader_1x06_P2.54mm_Horizontal, symbol Connector_Generic:Conn_01x06
- added LED1: DIGIT-A, LED_SMD:LED_SK6812_PLCC4_5.0x5.0mm_P3.2mm, symbol LED:SK6812
- added LED10: BL-2, LED_SMD:LED_SK6812_PLCC4_5.0x5.0mm_P3.2mm, symbol LED:SK6812
- added LED11: BL-3, LED_SMD:LED_SK6812_PLCC4_5.0x5.0mm_P3.2mm, symbol LED:SK6812
- added LED12: BL-4, LED_SMD:LED_SK6812_PLCC4_5.0x5.0mm_P3.2mm, symbol LED:SK6812
- added LED13: BL-5, LED_SMD:LED_SK6812_PLCC4_5.0x5.0mm_P3.2mm, symbol LED:SK6812
- added LED14: BL-6, LED_SMD:LED_SK6812_PLCC4_5.0x5.0mm_P3.2mm, symbol LED:SK6812
- added LED2: DIGIT-B, LED_SMD:LED_SK6812_PLCC4_5.0x5.0mm_P3.2mm, symbol LED:SK6812
- added LED3: DIGIT-C, LED_SMD:LED_SK6812_PLCC4_5.0x5.0mm_P3.2mm, symbol LED:SK6812
- added LED4: DIGIT-D, LED_SMD:LED_SK6812_PLCC4_5.0x5.0mm_P3.2mm, symbol LED:SK6812
- added LED5: DIGIT-E, LED_SMD:LED_SK6812_PLCC4_5.0x5.0mm_P3.2mm, symbol LED:SK6812
- added LED6: DIGIT-F, LED_SMD:LED_SK6812_PLCC4_5.0x5.0mm_P3.2mm, symbol LED:SK6812
- added LED7: DIGIT-G, LED_SMD:LED_SK6812_PLCC4_5.0x5.0mm_P3.2mm, symbol LED:SK6812
- added LED8: DIGIT-H, LED_SMD:LED_SK6812_PLCC4_5.0x5.0mm_P3.2mm, symbol LED:SK6812
- added LED9: BL-1, LED_SMD:LED_SK6812_PLCC4_5.0x5.0mm_P3.2mm, symbol LED:SK6812
Connections:
- new net: LED1.4 (DOUT), LED2.2 (DIN)
- new net: LED2.4 (DOUT), LED3.2 (DIN)
- new net: LED12.4 (DOUT), LED13.2 (DIN)
- new net: LED13.4 (DOUT), LED14.2 (DIN)
- new net: LED10.4 (DOUT), LED11.2 (DIN)
- new net: LED11.4 (DOUT), LED12.2 (DIN)
- new net: LED3.4 (DOUT), LED4.2 (DIN)
- new net: LED10.2 (DIN), LED9.4 (DOUT)
- new net: LED6.4 (DOUT), LED7.2 (DIN)
- new net: LED7.4 (DOUT), LED8.2 (DIN)
- new net: LED5.4 (DOUT), LED6.2 (DIN)
- new net: LED4.4 (DOUT), LED5.2 (DIN)
- new net +5V: C1.1, C10.1, C11.1, C12.1, C13.1, C14.1, C2.1, C3.1, C4.1, C5.1, C6.1, C7.1, C8.1, C9.1, D2.1 (K), D3.1 (K), LED1.3 (VDD), LED10.3 (VDD), LED11.3 (VDD), LED12.3 (VDD), LED13.3 (VDD), LED14.3 (VDD), LED2.3 (VDD), LED3.3 (VDD), LED4.3 (VDD), LED5.3 (VDD), LED6.3 (VDD), LED7.3 (VDD), LED8.3 (VDD), LED9.3 (VDD)
- new net BL_IN: J1.4 (Pin_4), LED9.2 (DIN)
- new net BL_OUT: J2.4 (Pin_4), LED14.4 (DOUT)
- new net DIGIT_IN: J1.3 (Pin_3), LED1.2 (DIN)
- new net DIGIT_OUT: J2.3 (Pin_3), LED8.4 (DOUT)
- new net GND: C1.2, C10.2, C11.2, C12.2, C13.2, C14.2, C2.2, C3.2, C4.2, C5.2, C6.2, C7.2, C8.2, C9.2, J1.5 (Pin_5), J1.6 (Pin_6), J2.5 (Pin_5), J2.6 (Pin_6), LED1.1 (VSS), LED10.1 (VSS), LED11.1 (VSS), LED12.1 (VSS), LED13.1 (VSS), LED14.1 (VSS), LED2.1 (VSS), LED3.1 (VSS), LED4.1 (VSS), LED5.1 (VSS), LED6.1 (VSS), LED7.1 (VSS), LED8.1 (VSS), LED9.1 (VSS)
- new net VCC_IN: D2.2 (A), J1.1 (Pin_1), J1.2 (Pin_2)
- new net VCC_OUT: D3.2 (A), J2.1 (Pin_1), J2.2 (Pin_2)
Other:
- note added: "Backlight LEDs"
- note added: "Board Interconnect"
- note added: "Main Segment LEDs"
- title: (none) -> Seven Segment Digit
